File: pcb/RP2350_80QFN_minimal.kicad_pcb (KiCad board)
At the start: 4 copper layers, 61 x 79 mm, 68 parts, among them J1 USB_C_Receptacle_USB2.0_14P, J2 XT30PW-M, J3 Conn_01x04_Pin, J4 SM03B-SRSS-TB, J5 TSW-116-08-G-T-RA, J6 Conn_01x04_Pin, J7 Conn_01x04_Pin, J8 Conn_Coaxial_Small, U1 RP2350_80QFN, U2 NCP1117-3.3_SOT223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

Commit message: RP Diode
Parts:
- added D4: SS56, SS56:SMB, F.Cu at (123.8, 115.8)
- added G***: LOGO, LOGO, F.Cu at (149.5, 71.1)
- added R16: 51.1k, Resistor_SMD:R_0805_2012Metric_Pad1.20x1.40mm_HandSolder, F.Cu at (133.0, 94.5)
- added R17: 23.7k, Resistor_SMD:R_0805_2012Metric_Pad1.20x1.40mm_HandSolder, F.Cu at (131.1, 100.9)
- added R18: 5k, Resistor_SMD:R_0805_2012Metric_Pad1.20x1.40mm_HandSolder, F.Cu at (134.4, 103.3)
- added R19: 23.7k, Resistor_SMD:R_0805_2012Metric_Pad1.20x1.40mm_HandSolder, F.Cu at (138.6, 99.6)
- added R20: 5k, Resistor_SMD:R_0805_2012Metric_Pad1.20x1.40mm_HandSolder, F.Cu at (138.6, 103.3)
- C25: value 10u -> 0.01u
- U6: value ~ -> TPS2121RUXR; footprint TPS22933ARSER:IC_RSE8 -> TPS2121RUXR:IC_TPS2121RUXR
- moved C25 9.61 mm to (129.6, 95.6), turned to 180 degrees
- moved C1 4.01 mm to (129.6, 97.9)
- moved U6 3.55 mm to (135.1, 99.3)
- moved G*** 2.47 mm to (151.6, 109.5)
- moved R5 0.66 mm to (130.2, 104.0)
- moved C4 0.64 mm to (141.3, 97.8)
Connections:
- C25 pad 1: Net-(U6-CAP) -> Net-(U6-SS)
- J2 pad P: Net-(U6-BAT) -> VBUS
- U6 pad 1: Net-(U6-BAT) -> VOUT
- U6 pad 2: USBV -> Net-(D4-PadC)
- U6 pad 3: VBUS -> GND
- U6 pad 4: GND -> Net-(U6-OV2)
- U6 pad 5: GND -> Net-(U6-OV1)
- U6 pad 6: Net-(U6-CAP) -> GND
- U6 pad 7: unconnected-(U6-VOUT-Pad7) -> USBV
Routing:
- net Net-(D4-PadC): track 0.00 -> 28.9 mm, vias 0 -> 4
- net Net-(U6-BAT): track 20.8 -> 0.00 mm, vias 2 -> 0
- net USBV: track 13.3 -> 23.9 mm, vias 0 -> 2
- net Net-(U6-OV1): track 0.00 -> 7.87 mm
- net Net-(U6-OV2): track 0.00 -> 7.80 mm
- net Net-(U6-ILIM): track 0.00 -> 6.48 mm
- net GND: track 48.8 -> 54.8 mm, vias 59 -> 63
- net Net-(U6-SS): track 0.00 -> 5.68 mm
- net Net-(U6-CAP): track 3.16 -> 0.00 mm
- net /GPIO21: track 52.2 -> 49.6 mm
- net VBUS: track 10.9 -> 13.3 mm, vias 2 -> 8
- net /SWCLK: track 45.0 -> 46.4 mm
- net VOUT: track 32.9 -> 33.5 mm
Other:
- board text added: "5v"
- board text removed: "3.3-12v"
- board text removed: "↑"
