File: pcb/_autosave-RP2350_80QFN_minimal.kicad_sch (KiCad schematic)
At the start: 66 parts, among them J1 USB_C_Receptacle_USB2.0_14P, J2 XT30PW-M, J3 Conn_01x04_Pin, J4 SM03B-SRSS-TB, J5 TSW-116-08-G-T-RA, J6 Conn_01x04_Pin, J7 Conn_01x04_Pin, J8 Conn_Coaxial_Small, SW1 SW_Push, SW2 SW_Push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

Commit message: RP Diode
Parts:
- removed J2: XT30PW-M, XT30PW-M:AMASS_XT30PW-M, symbol XT30PW-M:XT30PW-M
- removed U6: ~, TPS22933ARSER:IC_RSE8, symbol TPS22933ARSER:TPS22933ARSER
- added D4: SS56, SS56:SMB, symbol SS56:SS56
- added R16: 51.1k, Resistor_SMD:R_0805_2012Metric_Pad1.20x1.40mm_HandSolder, symbol Device:R
- added R17, R19: 23.7k, Resistor_SMD:R_0805_2012Metric_Pad1.20x1.40mm_HandSolder, symbol Device:R
- added R18, R20: 5k, Resistor_SMD:R_0805_2012Metric_Pad1.20x1.40mm_HandSolder, symbol Device:R
- added U6: TPS2121RUXR, TPS2121RUXR:IC_TPS2121RUXR, symbol TPS2121RUXR:TPS2121RUXR
- C25: value 10u -> 0.01u
Connections:
- net GND: now also R16.1, R18.1, R20.1, U6.12 (GND), U6.3 (CP2), U6.6 (PR1), U6.9 (ST)
- net USBV: now also R19.2, U6.7 (IN1), U6.7_1 (IN1)
- net VBUS: now also D4.A
- net VOUT: now also U6.1 (OUT), U6.1_1 (OUT), U6.8 (OUT), U6.8_1 (OUT)
- net at C25.1: now also U6.11 (SS)
- new net: R16.2, U6.10 (ILIM)
- new net: D4.C, R17.2, U6.2 (IN2), U6.2_1 (IN2)
- new net: R17.1, R18.2, U6.4 (OV2)
- new net: R19.1, R20.2, U6.5 (OV1)
